File: outputs/bat-module/bat-module.kicad_sch (KiCad schematic)
At the start: 0 parts

Commit message: hardware: reproducing eps2 schematics for battery monitoring
Parts:
- added C1, C2: 1000pF/50V, symbol Device:C
- added C3: 0.47uF/50V, symbol Device:C
- added C4, C5: 0.1uF/50V, symbol Device:C
- added D2: D_Schottky_Filled, symbol Device:D_Schottky_Filled
- added H1, H2, H3: MountingHole, MountingHole:MountingHole_3.2mm_M3_ISO14580_Pad, symbol Mechanical:MountingHole
- added H4: MountingHole_Pad, MountingHole:MountingHole_3.2mm_M3_ISO14580_Pad, symbol Mechanical:MountingHole_Pad
- added IC1: FDS6898AZ, SOIC127P600X175-8N, symbol FDS6898AZ-:FDS6898AZ
- added IC2: DS2777G+, SON40P500X300X80-15N-D, symbol DS2777G+:DS2777G+
- added R1: 1M, Resistor_SMD:R_0603_1608Metric_Pad0.98x0.95mm_HandSolder, symbol Device:R
- added R10, R11, R12, R8: 150R, symbol Device:R
- added R13, R14, R2: 0R, symbol Device:R
- added R3, R5, R6, R7, R9: 1K, symbol Device:R
- added R4: 470R, symbol Device:R
- added RSense1: 0.01R/0.5W, symbol Device:R
- added TP1: CC Test Point, symbol Connector:TestPoint
- added TP2: DC Test Point, symbol Connector:TestPoint
- added Z1, Z2: 3SMAJ5919B-TP, DIOM5226X244N, symbol 3SMAJ5919B-TP:3SMAJ5919B-TP
Connections:
- new net: IC1.4 (G1), R5.2, TP1.1
- new net: D2.1 (K), IC2.10 (PLS), R7.2
- new net: IC2.12 (SCL/OVD), R10.1
- new net: IC2.4 (VIN2), R3.2
- new net: C1.1, C2.1
- new net: C5.2, IC2.2 (VDD), R8.2
- new net: IC1.1 (S2), IC1.3 (S1), R4.1
- new net: IC2.1 (CC), R5.1
- new net: IC1.2 (G2), R6.1, TP2.1
- new net: IC2.3 (DC), R6.2
- new net: C3.2, IC2.14 (CP)
- new net: H4.1, R1.1
- new net: IC2.11 (SDA/DQ), R11.2, Z2.1 (K)
- new net: IC2.5 (VIN1), R9.1
- new net: C4.2, IC2.6 (VB)
- new net: IC2.9 (PIO), R12.2
- new net +VBat: C1.2, IC1.7 (D2_1), IC1.8 (D2_2), R2.2, R3.1, R8.1
- new net -VBat: C4.1, C5.1, R14.2
- new net GND: R1.2
- new net GNDREF: D2.2 (A), IC2.15 (EP), R13.1, Z1.2 (A), Z2.2 (A)
- new net I2C0_SCL: R10.2
- new net I2C0_SDA: R11.1
- new net PIO: R12.1, Z1.1 (K)
- new net SRC: C3.1, IC2.13 (SRC), R4.2
- new net VBat_Common: R9.2
- new net VCC: C2.2, IC1.5 (D1_1), IC1.6 (D1_2), R2.1, R7.1
- new net V_sense0_N: IC2.8 (SNS), R13.2, RSense1.1
- new net V_sense0_P: IC2.7 (VSS), R14.1, RSense1.2
Other:
- note added: "Battery Monitoring"
- note added: "Mechanical"
- note added: "PWR Flags"
