File: source/bat-module/bat-module.kicad_sch (KiCad schematic)
At the start: 31 parts, among them IC1 FDS6898AZ, IC2 DS2777G+

Commit message: hardware: moving main files
Other:
- added sheet batteries (batteries.kicad_sch)
Changed lines of the file:
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@@
+    )
+  )
+  (sheet (at 304.8 0) (size 12.7 204.47) (fields_autoplaced)
+    (stroke (width 0.1524) (type solid))
+    (fill (color 0 0 0 0.0000))
+    (property "Sheetname" "batteries" (at 304.8 -0.7116 0)
+      (effects (font (size 1.27 1.27)) (justify left bottom))
+    )
+    (property "Sheetfile" "batteries.kicad_sch" (at 304.8 205.0546 0)
+      (effects (font (size 1.27 1.27)) (justify left top))
+    )
+    (instances
+      (project "bat-module"
+        (path "/95270ebd-bf33-49a5-840f-dadc8a9f9793" (page "2"))
+      )
     )
   )
