File: bat-module.kicad_sch (KiCad schematic)
At the start: 10 parts, among them J3 Conn_01x02_Socket, J4 Conn_01x03_Socket, J5 Conn_01x04_Socket, J7 Conn_01x04_Socket

Commit message: general improvements in schematics
Parts:
- removed J4: Conn_01x03_Socket, Connector_Molex:Molex_PicoBlade_53048-0410_1x04_P1.25mm_Horizontal, symbol Connector:Conn_01x03_Socket
- removed J5: Conn_01x04_Socket, Connector_Molex:Molex_PicoBlade_53048-0410_1x04_P1.25mm_Horizontal, symbol Connector:Conn_01x04_Socket
- added J1: Conn_01x05_Socket, Connector_Molex:Molex_PicoBlade_53261-0571_1x05-1MP_P1.25mm_Horizontal, symbol Connector:Conn_01x05_Socket
- J3: footprint (none) -> footprints:CON_2053380002
- J5, J7: footprint (none) -> Connector_Molex:Molex_PicoBlade_53261-0471_1x04-1MP_P1.25mm_Horizontal
Connections:
- net GNDREF: now also J1.5 (Pin_5)
- net bat-monitoring/I2C0_SCL: now also J1.3 (Pin_3)
- net bat-monitoring/I2C0_SDA: now also J1.2 (Pin_2)
- net bat-monitoring/PIO: now also J1.4 (Pin_4)
- new net batteries/3V3_A_~{EN}: J1.1 (Pin_1)
Other:
- sheet bat-monitoring ports: added 3V3; removed none
- sheet batteries ports: added 3V3, 3V3_A_~{EN}; removed 5V0, 5V0_A_~{EN}
- sheet heater-circuit ports: added 3V3; removed 5V0
Changed lines of the file:
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@@
   (junction (at 69.596 45.72) (diameter 0) (color 0 0 0 0)
   )
-  (junction (at 50.8 173.99) (diameter 0) (color 0 0 0 0)
-  )
-  (junction (at 50.8 179.07) (diameter 0) (color 0 0 0 0)
-  )
-  (junction (at 50.8 176.53) (diameter 0) (color 0 0 0 0)
+  (junction (at 170.688 108.712) (diameter 0) (color 0 0 0 0)
   )
   (wire (pts (xy 52.578 50.8) (xy 69.596 50.8))
@@
     (stroke (width 0) (type default))
   )
+  (wire (pts (xy 90.678 149.606) (xy 166.116 149.606))
+    (stroke (width 0) (type default))
+  )
   (wire (pts (xy 50.8 173.99) (xy 81.156 173.99))
     (stroke (width 0) (type default))
@@
     (stroke (width 0) (type default))
   )
+  (wire (pts (xy 170.688 108.712) (xy 121.285 108.712))
+    (stroke (width 0) (type default))
+  )
   (wire (pts (xy 69.596 45.72) (xy 52.578 45.72))
     (stroke (width 0) (type default))
   )
+  (wire (pts (xy 170.688 108.712) (xy 189.23 108.712))
+    (stroke (width 0) (type default))
+  )
   (wire (pts (xy 69.596 50.8) (xy 69.596 45.72))
     (stroke (width 0) (type default))
@@
     (stroke (width 0) (type default))
   )
+  (wire (pts (xy 90.678 181.61) (xy 90.678 149.606))
+    (stroke (width 0) (type default))
+  )
   (wire (pts (xy 133.985 44.196) (xy 127 44.196))
     (stroke (width 0) (type default))
@@
     (stroke (width 0) (type default))
   )
-  (wire (pts (xy 170.688 65.405) (xy 170.688 88.646))
+  (wire (pts (xy 50.8 181.61) (xy 90.678 181.61))
+    (stroke (width 0) (type default))
+  )
+  (wire (pts (xy 170.688 65.405) (xy 170.688 108.712))
+    (stroke (width 0) (type default))
+  )
+  (wire (pts (xy 121.285 108.712) (xy 121.285 108.458))
     (stroke (width 0) (type default))
   )
@@
     (stroke (width 0) (type default))
   )
+  (wire (pts (xy 166.116 149.606) (xy 166.116 65.405))
+    (stroke (width 0) (type default))
+  )
   (wire (pts (xy 50.546 108.458) (xy 90.805 108.458))
     (stroke (width 0) (type default))
   )
   (wire (pts (xy 50.8 176.53) (xy 83.82 176.53))
-    (stroke (width 0) (type default))
-  )
-  (wire (pts (xy 170.688 88.646) (xy 189.23 88.646))
     (stroke (width 0) (type default))
   )
@@
       (effects (font (size 1.27 1.27)) (justify left))
     )
-    (property "Footprint" "" (at 45.466 108.458 0)
+    (property "Footprint" "footprints:CON_2053380002" (at 45.466 108.458 0)
       (effects (font (size 1.27 1.27)) hide)
     )
@@
         (path "/95270ebd-bf33-49a5-840f-dadc8a9f9793/b57b31e8-d0d5-445b-837b-f145ff19436b"
           (reference "J7") (unit 1)
+        )
+      )
+    )
+  )
+  (symbol (lib_id "Connector:Conn_01x05_Socket") (at 45.72 176.53 180) (unit 1)
+    (in_bom yes) (on_board yes) (dnp no) (fields_autoplaced)
+    (property "Reference" "J1" (at 46.355 166.37 0)
+      (effects (font (size 1.27 1.27)))
+    )
+    (property "Value" "Conn_01x05_Socket" (at 46.355 168.91 0)
+      (effects (font (size 1.27 1.27)))
+    )
+    (property "Footprint" "Connector_Molex:Molex_PicoBlade_53261-0571_1x05-1MP_P1.25mm_Horizontal" (at 45.72 176.53 0)
+      (effects (font (size 1.27 1.27)) hide)
+    )
+    (property "Datasheet" "~" (at 45.72 176.53 0)
+      (effects (font (size 1.27 1.27)) hide)
+    )
+    (pin "1")
+    (pin "2")
+    (pin "3")
+    (pin "4")
+    (pin "5")
+    (instances
+      (project "bat-module"
+        (path "/95270ebd-bf33-49a5-840f-dadc8a9f9793"
+          (reference "J1") (unit 1)
         )
       )
@@
     )
   )
-  (symbol (lib_id "Connector:Conn_01x03_Socket") (at 45.72 176.53 180) (unit 1)
-    (in_bom yes) (on_board yes) (dnp no) (fields_autoplaced)
-    (property "Reference" "J4" (at 44.45 177.8 0)
-      (effects (font (size 1.27 1.27)) (justify left) hide)
-    )
-    (property "Value" "Conn_01x03_Socket" (at 44.45 175.26 0)
-      (effects (font (size 1.27 1.27)) (justify left) hide)
-    )
-    (property "Footprint" "Connector_Molex:Molex_PicoBlade_53048-0410_1x04_P1.25mm_Horizontal" (at 45.72 176.53 0)
-      (effects (font (size 1.27 1.27)) hide)
-    )
-    (property "Datasheet" "~" (at 45.72 176.53 0)
-      (effects (font (size 1.27 1.27)) hide)
-    )
-    (pin "1")
-    (pin "2")
-    (pin "3")
-    (instances
-      (project "bat-module"
-        (path "/95270ebd-bf33-49a5-840f-dadc8a9f9793"
-          (reference "J4") (unit 1)
-        )
-        (path "/95270ebd-bf33-49a5-840f-dadc8a9f9793/b57b31e8-d0d5-445b-837b-f145ff19436b"
-          (reference "J8") (unit 1)
-        )
-      )
-    )
-  )
   (symbol (lib_id "Connector:Conn_01x04_Socket") (at 253.365 95.885 0) (unit 1)
     (in_bom yes) (on_board yes) (dnp no) (fields_autoplaced)
@@
       (effects (font (size 1.27 1.27)) (justify left))
     )
-    (property "Footprint" "" (at 253.365 95.885 0)
+    (property "Footprint" "Connector_Molex:Molex_PicoBlade_53261-0471_1x04-1MP_P1.25mm_Horizontal" (at 253.365 95.885 0)
       (effects (font (size 1.27 1.27)) hide)
     )
@@
     )
   )
-  (symbol (lib_id "Connector:Conn_01x04_Socket") (at 45.72 176.53 180) (unit 1)
-    (in_bom yes) (on_board yes) (dnp no) (fields_autoplaced)
-    (property "Reference" "J5" (at 44.45 176.53 0)
-      (effects (font (size 1.27 1.27)) (justify left))
-    )
-    (property "Value" "Conn_01x04_Socket" (at 44.45 173.99 0)
-      (effects (font (size 1.27 1.27)) (justify left))
-    )
-    (property "Footprint" "Connector_Molex:Molex_PicoBlade_53048-0410_1x04_P1.25mm_Horizontal" (at 45.72 176.53 0)
-      (effects (font (size 1.27 1.27)) hide)
-    )
-    (property "Datasheet" "~" (at 45.72 176.53 0)
-      (effects (font (size 1.27 1.27)) hide)
-    )
-    (pin "1")
-    (pin "2")
-    (pin "3")
-    (pin "4")
-    (instances
-      (project "bat-module"
-        (path "/95270ebd-bf33-49a5-840f-dadc8a9f9793"
-          (reference "J5") (unit 1)
-        )
-        (path "/95270ebd-bf33-49a5-840f-dadc8a9f9793/b57b31e8-d0d5-445b-837b-f145ff19436b"
-          (reference "J9") (unit 1)
-        )
-      )
-    )
-  )
   (symbol (lib_id "Mechanical:MountingHole") (at 145.796 171.196 0) (unit 1)
     (in_bom no) (on_board yes) (dnp no)
@@
       (effects (font (size 1.27 1.27)) (justify left))
     )
-    (property "Footprint" "" (at 47.498 48.26 0)
+    (property "Footprint" "Connector_Molex:Molex_PicoBlade_53261-0471_1x04-1MP_P1.25mm_Horizontal" (at 47.498 48.26 0)
       (effects (font (size 1.27 1.27)) hide)
     )
@@
       (effects (font (size 1.27 1.27)) (justify left top))
     )
-    (pin "5V0" output (at 189.23 88.646 180)
-      (effects (font (size 1.27 1.27)) (justify left))
-    )
     (pin "RTD3" input (at 219.71 95.885 0)
       (effects (font (size 1.27 1.27)) (justify right))
@@
     (pin "RTD6" input (at 219.71 98.425 0)
       (effects (font (size 1.27 1.27)) (justify right))
+    )
+    (pin "3V3" output (at 189.23 108.712 180)
+      (effects (font (size 1.27 1.27)) (justify left))
     )
     (instances
@@
       (effects (font (size 1.27 1.27)) (justify left top))
     )
-    (pin "5V0" output (at 170.688 65.405 270)
-      (effects (font (size 1.27 1.27)) (justify left))
-    )
-    (pin "5V0_A_~{EN}" input (at 176.53 48.768 0)
-      (effects (font (size 1.27 1.27)) (justify right))
-    )
     (pin "-VBat" input (at 133.985 48.006 180)
       (effects (font (size 1.27 1.27)) (justify left))
@@
     )
     (pin "+VBatB" input (at 133.985 39.37 180)
+      (effects (font (size 1.27 1.27)) (justify left))
+    )
+    (pin "3V3_A_~{EN}" input (at 166.116 65.405 270)
+      (effects (font (size 1.27 1.27)) (justify left))
+    )
+    (pin "3V3" output (at 170.688 65.405 270)
       (effects (font (size 1.27 1.27)) (justify left))
     )
@@
       (effects (font (size 1.27 1.27)) (justify right))
     )
+    (pin "3V3" output (at 121.285 108.458 0)
+      (effects (font (size 1.27 1.27)) (justify right))
+    )
