File: bat-monitoring.kicad_sch (KiCad schematic)
At the start: 27 parts, among them IC1 FDS6898AZ, IC2 DS2777G+

Commit message: general improvements in schematics
Parts:
- D2: footprint (none) -> footprints:NSVR0320MW2T1G; now left out of the parts list
- IC1: footprint lib:FDS6898AZ -> footprints:FDS6898AZ
- IC2: footprint lib:DS2777G+ -> footprints:DS2777G+
- R2: now left out of the parts list
- RSense1: footprint (none) -> Resistor_SMD:R_1206_3216Metric_Pad1.30x1.75mm_HandSolder
- TP1, TP2: footprint (none) -> TestPoint:TestPoint_Pad_D2.5mm
- Z1: footprint DIOM5226X244N -> footprints:3SMAJ5919B-TP
Connections:
- net +3V3: no longer R15.1, R16.1
- new net 3V3: R15.1, R16.1
Changed lines of the file:
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@@
     (effects (font (size 1.27 1.27)) (justify left))
+  )
+  (hierarchical_label "3V3" (shape output) (at 235.585 75.565 180) (fields_autoplaced)
+    (effects (font (size 1.27 1.27)) (justify right))
   )
   (hierarchical_label "Veps+" (shape input) (at 42.545 52.705 0) (fields_autoplaced)
@@
     (effects (font (size 1.27 1.27)) (justify left))
   )
+  (hierarchical_label "3V3" (shape output) (at 235.585 62.865 180) (fields_autoplaced)
+    (effects (font (size 1.27 1.27)) (justify right))
+  )
   (symbol (lib_id "Connector:TestPoint") (at 92.075 97.155 90) (unit 1)
     (in_bom yes) (on_board yes) (dnp no)
@@
       (effects (font (size 1.27 1.27)) (justify left))
     )
-    (property "Footprint" "" (at 92.075 92.075 0)
+    (property "Footprint" "TestPoint:TestPoint_Pad_D2.5mm" (at 92.075 92.075 0)
       (effects (font (size 1.27 1.27)) hide)
     )
@@
       (effects (font (size 1.27 1.27)))
     )
-    (property "Footprint" "lib:FDS6898AZ" (at 104.775 161.595 0)
+    (property "Footprint" "footprints:FDS6898AZ" (at 104.775 161.595 0)
       (effects (font (size 1.27 1.27)) (justify left top) hide)
     )
@@
       (effects (font (size 1.27 1.27)) (justify left))
     )
-    (property "Footprint" "" (at 99.695 102.235 0)
+    (property "Footprint" "TestPoint:TestPoint_Pad_D2.5mm" (at 99.695 102.235 0)
       (effects (font (size 1.27 1.27)) hide)
     )
@@
       (effects (font (size 1.27 1.27)))
     )
-    (property "Footprint" "lib:DS2777G+" (at 106.045 221.285 0)
+    (property "Footprint" "footprints:DS2777G+" (at 106.045 221.285 0)
       (effects (font (size 1.27 1.27)) (justify left top) hide)
     )
@@
   )
   (symbol (lib_id "Device:D_Schottky_Filled") (at 57.785 151.765 270) (unit 1)
-    (in_bom yes) (on_board yes) (dnp no)
+    (in_bom no) (on_board yes) (dnp no)
     (property "Reference" "D2" (at 53.975 153.035 90)
       (effects (font (size 1.27 1.27)) (justify left))
@@
       (effects (font (size 1.27 1.27)) (justify left))
     )
-    (property "Footprint" "" (at 57.785 151.765 0)
+    (property "Footprint" "footprints:NSVR0320MW2T1G" (at 57.785 151.765 0)
       (effects (font (size 1.27 1.27)) hide)
     )
@@
       (effects (font (size 1.27 1.27)) (justify left))
     )
-    (property "Footprint" "DIOM5226X244N" (at -59.995 154.305 0)
+    (property "Footprint" "footprints:3SMAJ5919B-TP" (at -59.995 154.305 0)
       (effects (font (size 1.27 1.27)) (justify left top) hide)
     )
@@
     )
   )
-  (symbol (lib_id "power:+3V3") (at 235.585 62.865 0) (unit 1)
-    (in_bom yes) (on_board yes) (dnp no) (fields_autoplaced)
-    (property "Reference" "#PWR08" (at 235.585 66.675 0)
-      (effects (font (size 1.27 1.27)) hide)
-    )
-    (property "Value" "+3V3" (at 235.585 57.785 0)
-      (effects (font (size 1.27 1.27)))
-    )
-    (property "Footprint" "" (at 235.585 62.865 0)
-      (effects (font (size 1.27 1.27)) hide)
-    )
-    (property "Datasheet" "" (at 235.585 62.865 0)
-      (effects (font (size 1.27 1.27)) hide)
-    )
-    (pin "1")
-    (instances
-      (project "bat-module"
-        (path "/95270ebd-bf33-49a5-840f-dadc8a9f9793"
-          (reference "#PWR08") (unit 1)
-        )
-        (path "/95270ebd-bf33-49a5-840f-dadc8a9f9793/b57b31e8-d0d5-445b-837b-f145ff19436b"
-          (reference "#PWR027") (unit 1)
-        )
-      )
-    )
-  )
   (symbol (lib_id "Device:C") (at 114.935 144.145 180) (unit 1)
     (in_bom yes) (on_board yes) (dnp no)
@@
       (effects (font (size 1.27 1.27)))
     )
-    (property "Footprint" "" (at 92.075 164.973 90)
+    (property "Footprint" "Resistor_SMD:R_1206_3216Metric_Pad1.30x1.75mm_HandSolder" (at 92.075 164.973 90)
       (effects (font (size 1.27 1.27)) hide)
     )
@@
         (path "/95270ebd-bf33-49a5-840f-dadc8a9f9793/b57b31e8-d0d5-445b-837b-f145ff19436b"
           (reference "C28") (unit 1)
-        )
-      )
-    )
-  )
-  (symbol (lib_id "power:+3V3") (at 235.585 75.565 0) (unit 1)
-    (in_bom yes) (on_board yes) (dnp no) (fields_autoplaced)
-    (property "Reference" "#PWR09" (at 235.585 79.375 0)
-      (effects (font (size 1.27 1.27)) hide)
-    )
-    (property "Value" "+3V3" (at 235.585 70.485 0)
-      (effects (font (size 1.27 1.27)))
-    )
-    (property "Footprint" "" (at 235.585 75.565 0)
-      (effects (font (size 1.27 1.27)) hide)
-    )
-    (property "Datasheet" "" (at 235.585 75.565 0)
-      (effects (font (size 1.27 1.27)) hide)
-    )
-    (pin "1")
-    (instances
-      (project "bat-module"
-        (path "/95270ebd-bf33-49a5-840f-dadc8a9f9793"
-          (reference "#PWR09") (unit 1)
-        )
-        (path "/95270ebd-bf33-49a5-840f-dadc8a9f9793/b57b31e8-d0d5-445b-837b-f145ff19436b"
-          (reference "#PWR030") (unit 1)
         )
       )
@@
   )
   (symbol (lib_id "Device:R") (at 95.885 55.245 90) (unit 1)
-    (in_bom yes) (on_board yes) (dnp no)
+    (in_bom no) (on_board yes) (dnp no)
     (property "Reference" "R2" (at 95.885 47.625 90)
       (effects (font (size 1.27 1.27)))
