File: batteries.kicad_sch (KiCad schematic)
At the start: 44 parts, among them J23 61300311121, Q28 EPC2016C, Q30 EPC2016C, Q9 SI2302DDS-T1-GE3, U30 LTC3833EUDC-TRPBF

Commit message: changing footprints and 3ds
Parts:
- C10, C20: footprint Capacitor_SMD:C_0603_1608Metric_Pad1.08x0.95mm_HandSolder -> footprints:C0603C104K5RACTU
- C12: footprint Capacitor_SMD:C_0603_1608Metric_Pad1.08x0.95mm_HandSolder -> footprints:C0603C332J5GACAUTO
- C14: footprint Capacitor_SMD:C_0603_1608Metric_Pad1.08x0.95mm_HandSolder -> footprints:C0603C101J5GACAUTO
- C16: footprint Capacitor_SMD:C_0603_1608Metric_Pad1.08x0.95mm_HandSolder -> footprints:C0603C102F3GACTU
- C22: footprint Capacitor_SMD:C_0603_1608Metric_Pad1.08x0.95mm_HandSolder -> footprints:GCM32ER71H475KA55L
- C24: footprint Capacitor_SMD:C_0603_1608Metric_Pad1.08x0.95mm_HandSolder -> footprints:T495X476K035ATE300
- C26, C28: footprint Capacitor_SMD:C_0603_1608Metric_Pad1.08x0.95mm_HandSolder -> footprints:C1210C106K5RACTU
- C30: footprint Capacitor_SMD:C_0603_1608Metric_Pad1.08x0.95mm_HandSolder -> footprints:C0805C105K5RACTU
- C32: footprint Capacitor_SMD:C_0603_1608Metric_Pad1.08x0.95mm_HandSolder -> footprints:C0603C220K5RACAUTO
- C34, C36, C38: footprint Capacitor_SMD:C_0603_1608Metric_Pad1.08x0.95mm_HandSolder -> footprints:GCM32ER71C226KE19L
- J23: footprint footprints:61300311121 -> footprints:three_position_jumper
- R34, R39: footprint Resistor_SMD:R_0603_1608Metric_Pad0.98x0.95mm_HandSolder -> footprints:CRCW0603100KFKEAHP
- R37: footprint Resistor_SMD:R_0603_1608Metric_Pad0.98x0.95mm_HandSolder -> footprints:CRCW060312K0FKEAHP
- R41: footprint Resistor_SMD:R_0603_1608Metric_Pad0.98x0.95mm_HandSolder -> footprints:CRCW060310R0FKEAHP
- R47: footprint Resistor_SMD:R_2010_5025Metric_Pad1.40x2.65mm_HandSolder -> footprints:WSL20108L000FEA18
- R50: footprint Resistor_SMD:R_0603_1608Metric_Pad0.98x0.95mm_HandSolder -> footprints:CRCW060390K9FKEAHP
- R52: footprint Resistor_SMD:R_0603_1608Metric_Pad0.98x0.95mm_HandSolder -> footprints:CRCW060320K0FKEAHP
- R76: footprint Resistor_SMD:R_0603_1608Metric_Pad0.98x0.95mm_HandSolder -> footprints:CRCW06030000Z0EAHP
- R96: footprint Resistor_SMD:R_0603_1608Metric_Pad0.98x0.95mm_HandSolder -> footprints:CRCW06032R20FKEAHP
- R97: footprint Resistor_SMD:R_0603_1608Metric_Pad0.98x0.95mm_HandSolder -> footprints:CRCW060382K0FKEA
Changed lines of the file:
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@@
       (effects (font (size 1.27 1.27)) (justify right))
     )
-    (property "Footprint" "Resistor_SMD:R_0603_1608Metric_Pad0.98x0.95mm_HandSolder" (at 334.772 100.584 0)
+    (property "Footprint" "footprints:CRCW060390K9FKEAHP" (at 334.772 100.584 0)
       (effects (font (size 1.27 1.27)) (justify left) hide)
     )
@@
       (effects (font (size 1.27 1.27)) (justify left))
     )
-    (property "Footprint" "Capacitor_SMD:C_0603_1608Metric_Pad1.08x0.95mm_HandSolder" (at 351.282 45.974 0)
+    (property "Footprint" "footprints:C0805C105K5RACTU" (at 351.282 45.974 0)
       (effects (font (size 1.27 1.27)) (justify left) hide)
     )
@@
       (effects (font (size 1.524 1.524)) (justify left))
     )
-    (property "Footprint" "Resistor_SMD:R_0603_1608Metric_Pad0.98x0.95mm_HandSolder" (at 216.662 146.304 0)
+    (property "Footprint" "footprints:CRCW06030000Z0EAHP" (at 216.662 146.304 0)
       (effects (font (size 1.27 1.27) italic) hide)
     )
@@
       (effects (font (size 1.27 1.27)) (justify right))
     )
-    (property "Footprint" "Resistor_SMD:R_0603_1608Metric_Pad0.98x0.95mm_HandSolder" (at 334.772 128.524 0)
+    (property "Footprint" "footprints:CRCW060320K0FKEAHP" (at 334.772 128.524 0)
       (effects (font (size 1.27 1.27)) (justify left) hide)
     )
@@
       (effects (font (size 1.27 1.27)))
     )
-    (property "Footprint" "Resistor_SMD:R_0603_1608Metric_Pad0.98x0.95mm_HandSolder" (at 182.372 80.264 0)
+    (property "Footprint" "footprints:CRCW0603100KFKEAHP" (at 182.372 80.264 0)
       (effects (font (size 1.27 1.27)) (justify left) hide)
     )
@@
       (effects (font (size 1.524 1.524)))
     )
-    (property "Footprint" "Resistor_SMD:R_0603_1608Metric_Pad0.98x0.95mm_HandSolder" (at 102.616 49.53 0)
+    (property "Footprint" "footprints:CRCW06032R20FKEAHP" (at 102.616 49.53 0)
       (effects (font (size 1.27 1.27) italic) hide)
     )
@@
       (effects (font (size 1.27 1.27)))
     )
-    (property "Footprint" "Resistor_SMD:R_0603_1608Metric_Pad0.98x0.95mm_HandSolder" (at 257.048 110.744 0)
+    (property "Footprint" "footprints:CRCW060310R0FKEAHP" (at 257.048 110.744 0)
       (effects (font (size 1.27 1.27)) (justify left) hide)
     )
@@
       (effects (font (size 1.27 1.27)) (justify left))
     )
-    (property "Footprint" "Capacitor_SMD:C_0603_1608Metric_Pad1.08x0.95mm_HandSolder" (at 170.942 99.314 0)
+    (property "Footprint" "footprints:C0603C332J5GACAUTO" (at 170.942 99.314 0)
       (effects (font (size 1.27 1.27)) (justify left) hide)
     )
@@
       (effects (font (size 1.27 1.27)))
     )
-    (property "Footprint" "Resistor_SMD:R_0603_1608Metric_Pad0.98x0.95mm_HandSolder" (at 257.048 119.634 0)
+    (property "Footprint" "footprints:CRCW060310R0FKEAHP" (at 257.048 119.634 0)
       (effects (font (size 1.27 1.27)) (justify left) hide)
     )
@@
       (effects (font (size 1.27 1.27)) (justify left))
     )
-    (property "Footprint" "Capacitor_SMD:C_0603_1608Metric_Pad1.08x0.95mm_HandSolder" (at 386.842 94.234 0)
+    (property "Footprint" "footprints:GCM32ER71C226KE19L" (at 386.842 94.234 0)
       (effects (font (size 1.27 1.27)) (justify left) hide)
     )
@@
       (effects (font (size 1.27 1.27)) (justify left))
     )
-    (property "Footprint" "Capacitor_SMD:C_0603_1608Metric_Pad1.08x0.95mm_HandSolder" (at 369.062 94.234 0)
+    (property "Footprint" "footprints:GCM32ER71C226KE19L" (at 369.062 94.234 0)
       (effects (font (size 1.27 1.27)) (justify left) hide)
     )
@@
       (effects (font (size 1.27 1.27)) (justify right))
     )
-    (property "Footprint" "Capacitor_SMD:C_0603_1608Metric_Pad1.08x0.95mm_HandSolder" (at 356.362 76.454 0)
+    (property "Footprint" "footprints:C0603C220K5RACAUTO" (at 356.362 76.454 0)
       (effects (font (size 1.27 1.27)) (justify left) hide)
     )
@@
       (effects (font (size 1.27 1.27)))
     )
-    (property "Footprint" "Resistor_SMD:R_2010_5025Metric_Pad1.40x2.65mm_HandSolder" (at 333.502 71.374 0)
+    (property "Footprint" "footprints:WSL20108L000FEA18" (at 333.502 71.374 0)
       (effects (font (size 1.27 1.27) italic) hide)
     )
@@
       (effects (font (size 1.27 1.27)) (justify right))
     )
-    (property "Footprint" "Capacitor_SMD:C_0603_1608Metric_Pad1.08x0.95mm_HandSolder" (at 253.492 65.024 0)
+    (property "Footprint" "footprints:C0603C104K5RACTU" (at 253.492 65.024 0)
       (effects (font (size 1.27 1.27)) (justify left) hide)
     )
@@
       (effects (font (size 1.27 1.27)) (justify left))
     )
-    (property "Footprint" "Capacitor_SMD:C_0603_1608Metric_Pad1.08x0.95mm_HandSolder" (at 343.662 45.974 0)
+    (property "Footprint" "footprints:C1210C106K5RACTU" (at 343.662 45.974 0)
       (effects (font (size 1.27 1.27)) (justify left) hide)
     )
@@
       (effects (font (size 1.27 1.27)) (justify left))
     )
-    (property "Footprint" "Resistor_SMD:R_0603_1608Metric_Pad0.98x0.95mm_HandSolder" (at 181.102 90.424 0)
+    (property "Footprint" "footprints:CRCW060312K0FKEAHP" (at 181.102 90.424 0)
       (effects (font (size 1.27 1.27)) (justify left) hide)
     )
@@
       (effects (font (size 1.27 1.27)))
     )
-    (property "Footprint" "Resistor_SMD:R_0603_1608Metric_Pad0.98x0.95mm_HandSolder" (at 240.538 68.834 0)
+    (property "Footprint" "footprints:CRCW060310R0FKEAHP" (at 240.538 68.834 0)
       (effects (font (size 1.27 1.27)) (justify left) hide)
     )
@@
       (effects (font (size 1.524 1.524)) (justify left))
     )
-    (property "Footprint" "Resistor_SMD:R_0603_1608Metric_Pad0.98x0.95mm_HandSolder" (at 334.772 105.664 0)
+    (property "Footprint" "footprints:CRCW06030000Z0EAHP" (at 334.772 105.664 0)
       (effects (font (size 1.27 1.27) italic) hide)
     )
@@
       (effects (font (size 1.27 1.27)) (justify left))
     )
-    (property "Footprint" "Capacitor_SMD:C_0603_1608Metric_Pad1.08x0.95mm_HandSolder" (at 181.102 99.314 0)
+    (property "Footprint" "footprints:C0603C101J5GACAUTO" (at 181.102 99.314 0)
       (effects (font (size 1.27 1.27)) (justify left) hide)
     )
@@
       (effects (font (size 1.27 1.27)) (justify left))
     )
-    (property "Footprint" "footprints:61300311121" (at 131.572 118.034 0)
+    (property "Footprint" "footprints:three_position_jumper" (at 131.572 118.034 0)
       (effects (font (size 1.27 1.27)) (justify left top) hide)
     )
@@
       (effects (font (size 1.27 1.27)) (justify left))
     )
-    (property "Footprint" "Capacitor_SMD:C_0603_1608Metric_Pad1.08x0.95mm_HandSolder" (at 115.062 70.104 0)
+    (property "Footprint" "footprints:C0603C104K5RACTU" (at 115.062 70.104 0)
       (effects (font (size 1.27 1.27)) (justify left) hide)
     )
@@
       (effects (font (size 1.27 1.27)) (justify left))
     )
-    (property "Footprint" "Capacitor_SMD:C_0603_1608Metric_Pad1.08x0.95mm_HandSolder" (at 191.262 99.314 0)
+    (property "Footprint" "footprints:C0603C102F3GACTU" (at 191.262 99.314 0)
       (effects (font (size 1.27 1.27)) (justify left) hide)
     )
@@
       (effects (font (size 1.27 1.27)) (justify left))
     )
-    (property "Footprint" "Capacitor_SMD:C_0603_1608Metric_Pad1.08x0.95mm_HandSolder" (at 267.462 70.104 0)
+    (property "Footprint" "footprints:GCM32ER71H475KA55L" (at 267.462 70.104 0)
       (effects (font (size 1.27 1.27)) (justify left) hide)
     )
@@
       (effects (font (size 1.27 1.27)) (justify left))
     )
-    (property "Footprint" "Capacitor_SMD:C_0603_1608Metric_Pad1.08x0.95mm_HandSolder" (at 322.072 45.974 0)
+    (property "Footprint" "footprints:T495X476K035ATE300" (at 322.072 45.974 0)
       (effects (font (size 1.27 1.27)) (justify left) hide)
     )
@@
       (effects (font (size 1.27 1.27)) (justify left))
     )
-    (property "Footprint" "Capacitor_SMD:C_0603_1608Metric_Pad1.08x0.95mm_HandSolder" (at 377.952 94.234 0)
+    (property "Footprint" "footprints:GCM32ER71C226KE19L" (at 377.952 94.234 0)
       (effects (font (size 1.27 1.27)) (justify left) hide)
     )
@@
       (effects (font (size 1.524 1.524)) (justify right))
     )
-    (property "Footprint" "Resistor_SMD:R_0603_1608Metric_Pad0.98x0.95mm_HandSolder" (at 169.672 99.314 0)
+    (property "Footprint" "footprints:CRCW060382K0FKEA" (at 169.672 99.314 0)
       (effects (font (size 1.27 1.27) italic) hide)
     )
@@
       (effects (font (size 1.27 1.27)) (justify right))
     )
-    (property "Footprint" "Resistor_SMD:R_0603_1608Metric_Pad0.98x0.95mm_HandSolder" (at 102.362 100.584 0)
+    (property "Footprint" "footprints:CRCW0603100KFKEAHP" (at 102.362 100.584 0)
       (effects (font (size 1.27 1.27)) (justify left) hide)
     )
@@
       (effects (font (size 1.27 1.27)) (justify left))
     )
-    (property "Footprint" "Capacitor_SMD:C_0603_1608Metric_Pad1.08x0.95mm_HandSolder" (at 332.232 45.974 0)
+    (property "Footprint" "footprints:C1210C106K5RACTU" (at 332.232 45.974 0)
       (effects (font (size 1.27 1.27)) (justify left) hide)
     )
@@
       (effects (font (size 1.524 1.524)) (justify left))
     )
-    (property "Footprint" "Resistor_SMD:R_0603_1608Metric_Pad0.98x0.95mm_HandSolder" (at 334.772 81.534 0)
+    (property "Footprint" "footprints:CRCW06030000Z0EAHP" (at 334.772 81.534 0)
       (effects (font (size 1.27 1.27) italic) hide)
     )
